File: KiCAD/_restore_backup_2026-07-14T18-33-41-810/Electrocardiograma.kicad_pcb (KiCad board)
At the start: 2 copper layers, 56.5 x 47.2 mm, 76 parts, among them J1 54-00174, J2 Conn_01x02_Pin, J3 USB_C_Receptacle_PowerOnly_6P, J4 Conn_01x02_Pin, J5 Conn_01x02_Pin, J6 Conn_01x04_Pin, U1 INA823DT, U2 ESP32-C3-WROOM-02, U3 TLV1117-33, U4 TLV4888, U5 TLV4888, U6 TLV1117-ADJ, U7 SC6038, U8 CH224K

Commit message: Vacaciones_Invierno Modulo De Carga
le añadimo modulo de carga a la placa, segun los chips que encontramos mas economicos, fue un leseo maomeno
Parts:
- moved R41 40.0 mm to (190.6, 72.0), turned to -90 degrees
- moved C15 4.78 mm to (153.0, 79.0), turned to 90 degrees
Connections:
- S1 pad SH1: -BATT_REG -> (no net)
- S1 pad SH2: -BATT_REG -> (no net)
Routing:
- net /Carga_Bateria: track 79.7 -> 22.9 mm, vias 1 -> 0
- net /Vbus: track 36.6 -> 22.5 mm, vias 2 -> 0
- net Net-(U7-CS): track 8.17 -> 0.00 mm
