File: KiCAD/_restore_backup_2026-07-14T18-33-41-810/Electrocardiograma.kicad_sch (KiCad schematic)
At the start: 80 parts, among them J1 54-00174, J2 Conn_01x02_Pin, J3 USB_C_Receptacle_PowerOnly_6P, J4 Conn_01x02_Pin, J5 Conn_01x02_Pin, J6 Conn_01x04_Pin, U1 INA823DT, U2 ESP32-C3-WROOM-02, U3 TLV1117-33, U4 TLV4888, U5 TLV4888, U6 TLV1117-ADJ, U7 SC6038, U8 CH224K

Commit message: Vacaciones_Invierno Modulo De Carga
le añadimo modulo de carga a la placa, segun los chips que encontramos mas economicos, fue un leseo maomeno
Connections:
- net -BATT_REG: no longer S1.SH1, S1.SH2
Changed lines of the file:
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@@
 	)
 	(junction
-		(at 304.8 34.29)
-		(diameter 0)
-		(color 0 0 0 0)
-	)
-	(junction
 		(at 290.83 63.5)
 		(diameter 0)
@@
 	(wire
 		(pts
-			(xy 304.8 36.83) (xy 303.53 36.83)
-		)
-		(stroke
-			(width 0)
-			(type default)
-		)
-	)
-	(wire
-		(pts
 			(xy 342.9 64.77) (xy 342.9 63.5)
 		)
@@
 	(wire
 		(pts
-			(xy 303.53 34.29) (xy 304.8 34.29)
-		)
-		(stroke
-			(width 0)
-			(type default)
-		)
-	)
-	(wire
-		(pts
 			(xy 72.39 257.81) (xy 72.39 270.51)
 		)
@@
 	(wire
 		(pts
-			(xy 304.8 34.29) (xy 304.8 36.83)
-		)
-		(stroke
-			(width 0)
-			(type default)
-		)
-	)
-	(wire
-		(pts
 			(xy 41.91 210.82) (xy 45.72 210.82)
 		)
@@
 	(wire
 		(pts
-			(xy 304.8 33.02) (xy 304.8 34.29)
-		)
-		(stroke
-			(width 0)
-			(type default)
-		)
-	)
-	(wire
-		(pts
 			(xy 46.99 99.06) (xy 69.85 99.06)
 		)
@@
 		(dnp no)
 		(property "Reference" "S1"
-			(at 296.164 43.688 0)
+			(at 295.91 35.56 0)
 			(show_name no)
 			(do_not_autoplace no)
@@
 		)
 		(property "Description" "12.9 x 9 x 5.6 mm, 4 mm Raised Slide Actuator, Right Angle, Through Hole, Slide Switch"
-			(at 295.91 50.292 0)
+			(at 295.91 43.18 0)
 			(hide yes)
 			(show_name no)
@@
 		)
 		(property "MF" "Same Sky"
-			(at 331.216 44.704 0)
+			(at 295.91 43.18 0)
 			(hide yes)
 			(show_name no)
@@
 		)
 		(property "MAXIMUM_PACKAGE_HEIGHT" "6.3mm"
-			(at 330.962 38.1 0)
+			(at 295.91 43.18 0)
 			(hide yes)
 			(show_name no)
@@
 		)
 		(property "Package" "Package"
-			(at 329.184 41.402 0)
+			(at 295.91 43.18 0)
 			(hide yes)
 			(show_name no)
@@
 		)
 		(property "Price" "None"
-			(at 318.516 40.386 0)
+			(at 295.91 43.18 0)
 			(hide yes)
 			(show_name no)
@@
 		)
 		(property "Check_prices" "https://www.snapeda.com/parts/SLW-129956-4A-RA-N-D/Same+Sky/view-part/?ref=eda"
-			(at 297.688 54.864 0)
+			(at 295.91 43.18 0)
 			(hide yes)
 			(show_name no)
@@
 		)
 		(property "STANDARD" "Manufacturer Recommendations"
-			(at 296.164 56.642 0)
+			(at 295.91 43.18 0)
 			(hide yes)
 			(show_name no)
@@
 		)
 		(property "PARTREV" "1.01"
-			(at 322.072 37.338 0)
+			(at 295.91 43.18 0)
 			(hide yes)
 			(show_name no)
@@
 		)
 		(property "SnapEDA_Link" "https://www.snapeda.com/parts/SLW-129956-4A-RA-N-D/Same+Sky/view-part/?ref=snap"
-			(at 296.926 52.578 0)
+			(at 295.91 43.18 0)
 			(hide yes)
 			(show_name no)
@@
 		)
 		(property "DigiKey" "SLW-129956-4A-RA-N-D"
-			(at 297.18 59.436 0)
+			(at 295.91 43.18 0)
 			(hide yes)
 			(show_name no)
@@
 		)
 		(property "Availability" "In Stock"
-			(at 325.882 33.528 0)
+			(at 295.91 43.18 0)
 			(hide yes)
 			(show_name no)
@@
 		)
 		(property "MANUFACTURER" "Same Sky"
-			(at 320.04 43.942 0)
+			(at 295.91 43.18 0)
 			(hide yes)
 			(show_name no)
@@
 		(pin "3"
 		)
-		(pin "SH2"
-		)
-		(pin "SH1"
-		)
 		(instances
 			(project "Electrocardiograma"
@@
 					(unit 1)
 				)
-			)
-		)
-	)
-	(symbol
-		(lib_id "power:-BATT")
-		(at 304.8 33.02 0)
-		(unit 1)
-		(body_style 1)
-		(exclude_from_sim no)
-		(in_bom yes)
-		(on_board yes)
-		(in_pos_files yes)
-		(dnp no)
-		(property "Reference" "#PWR041"
-			(at 304.8 36.83 0)
-			(hide yes)
-			(show_name no)
-			(do_not_autoplace no)
-			(effects
-				(font
-					(size 1.27 1.27)
-				)
-			)
-		)
-		(property "Value" "-BATT_REG"
-			(at 310.388 28.702 0)
-			(show_name no)
-			(do_not_autoplace no)
-			(effects
-				(font
-					(size 1.27 1.27)
-				)
-				(justify right)
-			)
-		)
-		(property "Footprint" ""
-			(at 304.8 33.02 0)
-			(hide yes)
-			(show_name no)
-			(do_not_autoplace no)
-			(effects
-				(font
-					(size 1.27 1.27)
-				)
-			)
-		)
-		(property "Datasheet" ""
-			(at 304.8 33.02 0)
-			(hide yes)
-			(show_name no)
-			(do_not_autoplace no)
-			(effects
-				(font
-					(size 1.27 1.27)
-				)
-			)
-		)
-		(property "Description" "Power symbol creates a global label with name \"-BATT\""
-			(at 304.8 33.02 0)
-			(hide yes)
-			(show_name no)
-			(do_not_autoplace no)
-			(effects
-				(font
-					(size 1.27 1.27)
-				)
-			)
-		)
-		(pin "1"
-		)
-		(instances
-			(project "Electrocardiograma"
-				(path "/daa88958-acc8-459e-83b6-465edaf551be"
-					(reference "#PWR041")
-					(unit 1)
-				)
