File: KiCAD/Electrocardiograma.kicad_sch (KiCad schematic)
At the start: 80 parts, among them J1 54-00174, J2 Conn_01x02_Pin, J3 USB_C_Receptacle_PowerOnly_6P, J4 Conn_01x02_Pin, J5 Conn_01x02_Pin, J6 Conn_01x04_Pin, U1 INA823DT, U2 ESP32-C3-WROOM-02, U3 TLV1117-33, U4 TLV4888, U5 TLV4888, U6 TLV1117-ADJ, U7 SC6038, U8 CH224K

Commit message: Final Details
Parts:
- added R44: 10k, Resistor_SMD:R_0805_2012Metric_Pad1.20x1.40mm_HandSolder, symbol Device:R
- R33: value 10 -> 47
Connections:
- net Vbus: now also R44.1
- net at U8.8 (VBUS): now also R44.2
Other:
- moved on the sheet: C17
Changed lines of the file:
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@@
 	)
 	(junction
-		(at 289.56 101.6)
-		(diameter 0)
-		(color 0 0 0 0)
-	)
-	(junction
 		(at 257.81 72.39)
 		(diameter 0)
@@
 	)
 	(junction
-		(at 304.8 123.19)
-		(diameter 0)
-		(color 0 0 0 0)
-	)
-	(junction
 		(at 74.93 71.12)
 		(diameter 0)
@@
 	)
 	(junction
+		(at 304.8 123.19)
+		(diameter 0)
+		(color 0 0 0 0)
+	)
+	(junction
 		(at 80.01 224.79)
 		(diameter 0)
@@
 	)
 	(junction
+		(at 289.56 101.6)
+		(diameter 0)
+		(color 0 0 0 0)
+	)
+	(junction
 		(at 316.23 63.5)
 		(diameter 0)
@@
 	)
 	(junction
+		(at 289.56 92.71)
+		(diameter 0)
+		(color 0 0 0 0)
+	)
+	(junction
 		(at 134.62 127)
 		(diameter 0)
@@
 	(wire
 		(pts
+			(xy 280.67 92.71) (xy 289.56 92.71)
+		)
+		(stroke
+			(width 0)
+			(type default)
+		)
+	)
+	(wire
+		(pts
 			(xy 378.46 105.41) (xy 373.38 105.41)
 		)
@@
 	(wire
 		(pts
-			(xy 304.8 123.19) (xy 316.23 123.19)
+			(xy 304.8 123.19) (xy 314.96 123.19)
 		)
 		(stroke
@@
 	(wire
 		(pts
-			(xy 316.23 121.92) (xy 316.23 123.19)
+			(xy 314.96 120.65) (xy 314.96 123.19)
 		)
 		(stroke
@@
 	(wire
 		(pts
+			(xy 280.67 102.87) (xy 280.67 100.33)
+		)
+		(stroke
+			(width 0)
+			(type default)
+		)
+	)
+	(wire
+		(pts
 			(xy 261.62 163.83) (xy 261.62 171.45)
 		)
@@
 	(wire
 		(pts
-			(xy 316.23 114.3) (xy 316.23 101.6)
+			(xy 314.96 113.03) (xy 314.96 101.6)
 		)
 		(stroke
@@
 	(wire
 		(pts
+			(xy 280.67 102.87) (xy 287.02 102.87)
+		)
+		(stroke
+			(width 0)
+			(type default)
+		)
+	)
+	(wire
+		(pts
 			(xy 275.59 43.18) (xy 281.94 43.18)
 		)
@@
 	(wire
 		(pts
-			(xy 289.56 101.6) (xy 316.23 101.6)
+			(xy 289.56 101.6) (xy 314.96 101.6)
 		)
 		(stroke
@@
 	)
 	(symbol
+		(lib_id "power:+3.3V")
+		(at 300.99 92.71 0)
+		(unit 1)
+		(body_style 1)
+		(exclude_from_sim no)
+		(in_bom yes)
+		(on_board yes)
+		(in_pos_files yes)
+		(dnp no)
+		(fields_autoplaced yes)
+		(property "Reference" "#PWR042"
+			(at 300.99 96.52 0)
+			(hide yes)
+			(show_name no)
+			(do_not_autoplace no)
+			(effects
+				(font
+					(size 1.27 1.27)
+				)
+			)
+		)
+		(property "Value" "+3.3V"
+			(at 300.99 87.63 0)
+			(show_name no)
+			(do_not_autoplace no)
+			(effects
+				(font
+					(size 1.27 1.27)
+				)
+			)
+		)
+		(property "Footprint" ""
+			(at 300.99 92.71 0)
+			(hide yes)
+			(show_name no)
+			(do_not_autoplace no)
+			(effects
+				(font
+					(size 1.27 1.27)
+				)
+			)
+		)
+		(property "Datasheet" ""
+			(at 300.99 92.71 0)
+			(hide yes)
+			(show_name no)
+			(do_not_autoplace no)
+			(effects
+				(font
+					(size 1.27 1.27)
+				)
+			)
+		)
+		(property "Description" "Power symbol creates a global label with name \"+3.3V\""
+			(at 300.99 92.71 0)
+			(hide yes)
+			(show_name no)
+			(do_not_autoplace no)
+			(effects
+				(font
+					(size 1.27 1.27)
+				)
+			)
+		)
+		(pin "1"
+		)
+		(instances
+			(project "Electrocardiograma"
+				(path "/daa88958-acc8-459e-83b6-465edaf551be"
+					(reference "#PWR042")
+					(unit 1)
+				)
+			)
+		)
+	)
+	(symbol
 		(lib_id "power:-BATT")
 		(at 281.94 227.33 0)
@@
 	)
 	(symbol
+		(lib_id "Device:R")
+		(at 280.67 96.52 0)
+		(mirror y)
+		(unit 1)
+		(body_style 1)
+		(exclude_from_sim no)
+		(in_bom yes)
+		(on_board yes)
+		(in_pos_files yes)
+		(dnp no)
+		(property "Reference" "R44"
+			(at 278.13 95.2499 0)
+			(show_name no)
+			(do_not_autoplace no)
+			(effects
+				(font
+					(size 1.27 1.27)
+				)
+				(justify left)
+			)
+		)
+		(property "Value" "10k"
+			(at 278.13 97.7899 0)
+			(show_name no)
+			(do_not_autoplace no)
+			(effects
+				(font
+					(size 1.27 1.27)
+				)
+				(justify left)
+			)
+		)
+		(property "Footprint" "Resistor_SMD:R_0805_2012Metric_Pad1.20x1.40mm_HandSolder"
+			(at 282.448 96.52 90)
+			(hide yes)
+			(show_name no)
+			(do_not_autoplace no)
+			(effects
+				(font
+					(size 1.27 1.27)
+				)
+			)
+		)
+		(property "Datasheet" ""
+			(at 280.67 96.52 0)
+			(hide yes)
+			(show_name no)
+			(do_not_autoplace no)
+			(effects
+				(font
+					(size 1.27 1.27)
+				)
+			)
+		)
+		(property "Description" "Resistor"
+			(at 280.67 96.52 0)
+			(hide yes)
+			(show_name no)
+			(do_not_autoplace no)
+			(effects
+				(font
+					(size 1.27 1.27)
+				)
+			)
+		)
+		(property "DigiKey" "P100KDACT-ND"
+			(at 280.67 96.52 90)
+			(hide yes)
+			(show_name no)
+			(do_not_autoplace no)
+			(effects
+				(font
+					(size 1.27 1.27)
+				)
+			)
+		)
+		(pin "1"
+		)
+		(pin "2"
+		)
+		(instances
+			(project "Electrocardiograma"
+				(path "/daa88958-acc8-459e-83b6-465edaf551be"
+					(reference "R44")
+					(unit 1)
+				)
+			)
+		)
+	)
+	(symbol
 		(lib_name "R_5")
 		(lib_id "Device:R")
@@
 			)
 		)
-		(property "Value" "10"
+		(property "Value" "47"
 			(at 284.48 222.2499 0)
 			(show_name no)
@@
 		(lib_name "C_Polarized_US_1")
 		(lib_id "Device:C_Polarized_US")
-		(at 316.23 118.11 0)
+		(at 314.96 116.84 0)
 		(unit 1)
 		(body_style 1)
@@
 		(fields_autoplaced yes)
 		(property "Reference" "C17"
-			(at 320.04 116.2049 0)
+			(at 318.77 114.9349 0)
 			(show_name no)
 			(do_not_autoplace no)
@@
 		)
 		(property "Value" "10uF"
-			(at 320.04 118.7449 0)
+			(at 318.77 117.4749 0)
 			(show_name no)
 			(do_not_autoplace no)
@@
 		)
 		(property "Footprint" "Capacitor_SMD:C_0805_2012Metric_Pad1.18x1.45mm_HandSolder"
-			(at 316.23 118.11 0)
+			(at 314.96 116.84 0)
 			(hide yes)
 			(show_name no)
@@
 		)
 		(property "Datasheet" ""
-			(at 316.23 118.11 0)
+			(at 314.96 116.84 0)
 			(hide yes)
 			(show_name no)
@@
 		)
 		(property "Description" "Polarized capacitor, US symbol"
-			(at 316.23 118.11 0)
+			(at 314.96 116.84 0)
 			(hide yes)
 			(show_name no)
@@
 		)
 		(property "DigiKey" "1276-1096-1-ND"
-			(at 316.23 118.11 0)
+			(at 314.96 116.84 0)
 			(hide yes)
 			(show_name no)

Commit message: Extra
Parts:
- C14: value 10u -> 10uF; DigiKey 490-1642-1-ND -> 1276-1096-1-ND
Changed lines of the file:
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@@
 			)
 		)
-		(property "Value" "10u"
+		(property "Value" "10uF"
 			(at 113.03 108.7764 90)
 			(show_name no)
@@
 			)
 		)
-		(property "DigiKey" "490-1642-1-ND"
+		(property "DigiKey" "1276-1096-1-ND"
 			(at 113.03 113.03 90)
 			(hide yes)

Commit message: Compra de Componentes atrasados
Cambio de resistencia para CH224
Parts:
- removed R42: 1k, Resistor_SMD:R_0805_2012Metric_Pad1.20x1.40mm_HandSolder, symbol Device:R
Connections:
- net +3.3V: now also C17.1, U8.1 (VDD)
Changed lines of the file:
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@@
 	)
 	(junction
-		(at 289.56 92.71)
-		(diameter 0)
-		(color 0 0 0 0)
-	)
-	(junction
 		(at 134.62 127)
 		(diameter 0)
@@
 	(symbol
 		(lib_id "power:+3.3V")
-		(at 300.99 92.71 0)
+		(at 289.56 100.33 0)
 		(unit 1)
 		(body_style 1)
@@
 		(fields_autoplaced yes)
 		(property "Reference" "#PWR042"
-			(at 300.99 96.52 0)
+			(at 289.56 104.14 0)
 			(hide yes)
 			(show_name no)
@@
 		)
 		(property "Value" "+3.3V"
-			(at 300.99 87.63 0)
+			(at 289.56 95.25 0)
 			(show_name no)
 			(do_not_autoplace no)
@@
 		)
 		(property "Footprint" ""
-			(at 300.99 92.71 0)
+			(at 289.56 100.33 0)
 			(hide yes)
 			(show_name no)
@@
 		)
 		(property "Datasheet" ""
-			(at 300.99 92.71 0)
+			(at 289.56 100.33 0)
 			(hide yes)
 			(show_name no)
@@
 		)
 		(property "Description" "Power symbol creates a global label with name \"+3.3V\""
-			(at 300.99 92.71 0)
+			(at 289.56 100.33 0)
 			(hide yes)
 			(show_name no)
@@
 					(unit 1)
 				)
-			)
-		)
-	)
-	(symbol
-		(lib_id "Device:R")
-		(at 289.56 96.52 0)
-		(unit 1)
-		(body_style 1)
-		(exclude_from_sim no)
-		(in_bom yes)
-		(on_board yes)
-		(in_pos_files yes)
-		(dnp no)
-		(fields_autoplaced yes)
-		(property "Reference" "R42"
-			(at 292.1 95.2499 0)
-			(show_name no)
-			(do_not_autoplace no)
-			(effects
-				(font
-					(size 1.27 1.27)
-				)
-				(justify left)
-			)
-		)
-		(property "Value" "1k"
-			(at 292.1 97.7899 0)
-			(show_name no)
-			(do_not_autoplace no)
-			(effects
-				(font
-					(size 1.27 1.27)
-				)
-				(justify left)
-			)
-		)
-		(property "Footprint" "Resistor_SMD:R_0805_2012Metric_Pad1.20x1.40mm_HandSolder"
-			(at 287.782 96.52 90)
-			(hide yes)
-			(show_name no)
-			(do_not_autoplace no)
-			(effects
-				(font
-					(size 1.27 1.27)
-				)
-			)
-		)
-		(property "Datasheet" ""
-			(at 289.56 96.52 0)
-			(hide yes)
-			(show_name no)
-			(do_not_autoplace no)
-			(effects
-				(font
-					(size 1.27 1.27)
-				)
-			)
-		)
-		(property "Description" "Resistor"
-			(at 289.56 96.52 0)
-			(hide yes)
-			(show_name no)
-			(do_not_autoplace no)
-			(effects
-				(font
-					(size 1.27 1.27)
-				)
-			)
-		)
-		(property "DigiKey" "P100KDACT-ND"
-			(at 289.56 96.52 90)
-			(hide yes)
-			(show_name no)
-			(do_not_autoplace no)
-			(effects
-				(font
-					(size 1.27 1.27)
-				)
-			)
-		)
-		(pin "1"
-		)
-		(pin "2"
-		)
-		(instances
-			(project "Electrocardiograma"
-				(path "/daa88958-acc8-459e-83b6-465edaf551be"
-					(reference "R42")
-					(unit 1)
-				)

Commit message: ih
Connections:
- net at J1.1: now also U1.2 (-); no longer U1.3 (+)
- net at J1.3: now also U1.3 (+); no longer U1.2 (-)
Other:
- note added: "Se cambia el TLV1117 por AMS1117 debido a que no se necesita bajo ruido para el ESP32"
Changed lines of the file:
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@@
+		)
+	)
+	(text "Se cambia el TLV1117 por AMS1117\ndebido a que no se necesita \nbajo ruido para el ESP32"
+		(exclude_from_sim no)
+		(at 333.248 55.626 0)
+		(effects
+			(font
+				(size 1.27 1.27)
+			)
 		)
 	)
@@
 	(wire
 		(pts
-			(xy 54.61 33.02) (xy 104.14 33.02)
-		)
-		(stroke
-			(width 0)
-			(type default)
-		)
-	)
-	(wire
-		(pts
 			(xy 127 43.18) (xy 127 36.83)
 		)
@@
 	(wire
 		(pts
+			(xy 54.61 35.56) (xy 91.44 35.56)
+		)
+		(stroke
+			(width 0)
+			(type default)
+		)
+	)
+	(wire
+		(pts
 			(xy 36.83 222.25) (xy 41.91 222.25)
 		)
@@
 	(wire
 		(pts
+			(xy 104.14 35.56) (xy 95.25 35.56)
+		)
+		(stroke
+			(width 0)
+			(type default)
+		)
+	)
+	(wire
+		(pts
 			(xy 303.53 43.18) (xy 313.69 43.18)
 		)
@@
 	(wire
 		(pts
+			(xy 91.44 35.56) (xy 91.44 33.02)
+		)
+		(stroke
+			(width 0)
+			(type default)
+		)
+	)
+	(wire
+		(pts
 			(xy 64.77 161.29) (xy 59.69 161.29)
 		)
@@
 	(wire
 		(pts
+			(xy 91.44 33.02) (xy 104.14 33.02)
+		)
+		(stroke
+			(width 0)
+			(type default)
+		)
+	)
+	(wire
+		(pts
 			(xy 353.06 43.18) (xy 358.14 43.18)
 		)
@@
 	(wire
 		(pts
-			(xy 54.61 35.56) (xy 104.14 35.56)
-		)
-		(stroke
-			(width 0)
-			(type default)
-		)
-	)
-	(wire
-		(pts
 			(xy 280.67 102.87) (xy 287.02 102.87)
 		)
@@
 	(wire
 		(pts
+			(xy 95.25 35.56) (xy 95.25 34.29)
+		)
+		(stroke
+			(width 0)
+			(type default)
+		)
+	)
+	(wire
+		(pts
 			(xy 341.63 100.33) (xy 336.55 100.33)
 		)
@@
 	(wire
 		(pts
+			(xy 54.61 34.29) (xy 54.61 33.02)
+		)
+		(stroke
+			(width 0)
+			(type default)
+		)
+	)
+	(wire
+		(pts
 			(xy 381 50.8) (xy 386.08 50.8)
 		)
@@
 		(pts
 			(xy 64.77 161.29) (xy 64.77 173.99)
+		)
+		(stroke
+			(width 0)
+			(type default)
+		)
+	)
+	(wire
+		(pts
+			(xy 54.61 34.29) (xy 95.25 34.29)
 		)
 		(stroke
@@
 	)
 	(label "To_ESP32"
-		(at 298.45 179.07 180)
+		(at 298.45 179.07 0)
 		(effects
 			(font
 				(size 1.27 1.27)
 			)
-			(justify right bottom)
-		)
-	)
+			(justify left bottom)
+		)
+	)

Commit message: Corrección opamp
Corregido un opamp mal trazado en el esquematico y pcb
Connections:
- net GND: now also U5.12 (+); no longer U5.13 (-)
- net at R12.2, R25.1: now also U5.13 (-); no longer U5.12 (+)
Changed lines of the file:
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@@
 	(wire
 		(pts
-			(xy 59.69 270.51) (xy 60.96 270.51)
-		)
-		(stroke
-			(width 0)
-			(type default)
-		)
-	)
-	(wire
-		(pts
 			(xy 335.28 43.18) (xy 337.82 43.18)
 		)
@@
 		(lib_id "Amplifier_Operational:TL074")
 		(at 62.23 270.51 0)
+		(mirror x)
 		(unit 4)
 		(body_style 1)
@@
 		(in_pos_files yes)
 		(dnp no)
-		(fields_autoplaced yes)
 		(property "Reference" "U5"
-			(at 62.23 260.35 0)
+			(at 62.23 280.67 0)
 			(show_name no)
 			(do_not_autoplace no)
@@
 		)
 		(property "Value" "TLV4888"
-			(at 62.23 262.89 0)
+			(at 62.23 278.13 0)
 			(show_name no)
 			(do_not_autoplace no)
@@
 		)
 		(property "Footprint" "Package_SO:SOIC-14_3.9x8.7mm_P1.27mm"
-			(at 60.96 267.97 0)
+			(at 60.96 273.05 0)
 			(hide yes)
 			(show_name no)
@@
 		)
 		(property "Datasheet" "http://www.ti.com/lit/ds/symlink/tl071.pdf"
-			(at 63.5 265.43 0)
+			(at 63.5 275.59 0)
 			(hide yes)
 			(show_name no)

Commit message: Added Charging indicator LED
Parts:
- added D6: LED, LED_SMD:LED_1206_3216Metric_Pad1.42x1.75mm_HandSolder, symbol Device:LED
- added R42: 470, Resistor_SMD:R_0805_2012Metric_Pad1.20x1.40mm_HandSolder, symbol Device:R
Connections:
- net -BATT_REG: now also R42.2
- net at U7.3 (CHRG): now also D6.2 (A)
- new net: D6.1 (K), R42.1
