File: KiCAD/Electrocardiograma.kicad_sch (KiCad schematic)
At the start: 89 parts, among them J1 54-00174, J2 Conn_01x02_Pin, J3 USB_C_Receptacle_PowerOnly_6P, J4 Conn_01x02_Pin, J5 Conn_01x02_Pin, J6 Conn_01x04_Pin, U1 INA823DT, U2 ESP32-C3-WROOM-02, U3 TLV1117-33, U4 TLV4888, U5 TLV4888, U6 TLV1117-ADJ, U7 SC6038, U8 CH224K

Commit message: Orden y purga de simulaciónes, ademas se añadieron las footprints faltantes
Parts:
- C20, C21, C22, C23, C24, C25: footprint (none) -> Capacitor_SMD:C_0805_2012Metric_Pad1.18x1.45mm_HandSolder
- D2: footprint Diode_SMD:D_SMA_Handsoldering -> Diode_SMD:D_SMA
Changed lines of the file:
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@@
 			)
 		)
-		(property "Footprint" ""
+		(property "Footprint" "Capacitor_SMD:C_0805_2012Metric_Pad1.18x1.45mm_HandSolder"
 			(at 187.96 240.9952 0)
 			(hide yes)
@@
 			)
 		)
-		(property "Footprint" ""
+		(property "Footprint" "Capacitor_SMD:C_0805_2012Metric_Pad1.18x1.45mm_HandSolder"
 			(at 110.7948 226.06 0)
 			(hide yes)
@@
 			)
 		)
-		(property "Footprint" ""
+		(property "Footprint" "Capacitor_SMD:C_0805_2012Metric_Pad1.18x1.45mm_HandSolder"
 			(at 186.69 317.8048 0)
 			(hide yes)
@@
 			)
 		)
-		(property "Footprint" ""
+		(property "Footprint" "Capacitor_SMD:C_0805_2012Metric_Pad1.18x1.45mm_HandSolder"
 			(at 146.05 109.5248 0)
 			(hide yes)
@@
 			)
 		)
-		(property "Footprint" ""
+		(property "Footprint" "Capacitor_SMD:C_0805_2012Metric_Pad1.18x1.45mm_HandSolder"
 			(at 131.1148 279.4 0)
 			(hide yes)
@@
 			)
 		)
-		(property "Footprint" "Diode_SMD:D_SMA_Handsoldering"
+		(property "Footprint" "Diode_SMD:D_SMA"
 			(at 464.82 70.485 0)
 			(hide yes)
@@
 			)
 		)
-		(property "Footprint" ""
+		(property "Footprint" "Capacitor_SMD:C_0805_2012Metric_Pad1.18x1.45mm_HandSolder"
 			(at 120.9548 339.09 0)
 			(hide yes)

Commit message: Schematic Adjustments
Parts:
- added R45, R47, R48, R49: 120, Resistor_SMD:R_0805_2012Metric_Pad1.20x1.40mm_HandSolder, symbol Device:R
- C26: footprint (none) -> Capacitor_SMD:C_0805_2012Metric_Pad1.18x1.45mm_HandSolder
Connections:
- net HPF_out: now also R45.2; no longer C20.2, R14.2, R17.2, U5.1
- net LPF_out: now also R48.2; no longer C11.2, C23.2, R21.2, U5.8
- net N50Hz_out: now also R47.2; no longer C21.2, C5.1, C8.1, R10.2, U5.7
- net Sensing_Out: now also R49.2; no longer C24.2, R25.2, U5.14
- new net: C21.2, C5.1, C8.1, R10.2, R47.1, U5.7
- new net: C20.2, R14.2, R17.2, R45.1, U5.1
- new net: C11.2, C23.2, R21.2, R48.1, U5.8
- new net: C24.2, R25.2, R49.1, U5.14
Other:
- moved on the sheet: C16

Commit message: diseño capacitores Cf
Parts:
- R17, R21: value 27K -> 2K7
- R19, R20, R22, R23: value 100K -> 10K
Other:
- note added: "C_f=10nF como filtro pasa bajos profuce una frecuencia de corte de F_c=5.9[kHz]"
- note added: "C_f=2.5nF Como cota inferior del filtro pasa bajos F_c=23.6[kHz] --> Media geometrica entre 1600Hz y 350kHz"
- note added: "C_f=3.7nF para aplanar la respuesta de C_i=1nF parasito"
- note added: "CriticamenteFiltrado"
- note added: "R=100[k] C=10[nF] F_c=159[Hz] R=10[k] C=10[nF] F_c=1591[Hz]"
- note added: "SobreFiltrado"
- note added: "SubFiltrado"
- note removed: "Hay que discutir sobre bajar el valor de resistencias de 100k y 26k7 del lazo de realimentación"
- moved on the sheet: C10, C11, C12, C13, C14, C20, C21, C22, C23, C24, C5, C6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

Commit message: .
Parts:
- added C27, C28, C29, C30: 10nF, Capacitor_SMD:C_0805_2012Metric_Pad1.18x1.45mm_HandSolder, symbol Device:C
Connections:
- net GND: now also C27.1, C28.1, C29.1, C30.1
- net HPF_out: now also C27.2
- net LPF_out: now also C29.2
- net N50Hz_out: now also C28.2
- net Sensing_Out: now also C30.2
Other:
- note added: "Entre Etapas"
- note added: "F_c=133[kHz] frecuencia de corte filtro pasa bajos pasivo RC"

Commit message: cambios de placa y esquematico
Parts:
- added C31: 10nF, Capacitor_SMD:C_0805_2012Metric_Pad1.18x1.45mm_HandSolder, symbol Device:C
- added R50: 120, Resistor_SMD:R_0805_2012Metric_Pad1.20x1.40mm_HandSolder, symbol Device:R
- R10: value 22K -> 2K67; DigiKey P22KDACT-ND -> (none)
- R11: value 33K -> 4k; DigiKey P33KDACT-ND -> (none)
- R12: DigiKey P100KDACT-ND -> (none)
- R17: value 2K7 -> 2K67; DigiKey 311-26.7KCRCT-ND -> (none)
- R21: value 2K7 -> 2K67
- R24: value 33K -> 1K
- R34: value 100K -> 1K
- R36: value 100K -> 1K; DigiKey P100KDACT-ND -> (none)
- R4: value 330k -> 33k
Connections:
- net GND: now also C31.1
- net Leveled_Signal: now also C31.2, R50.2; no longer C22.1, R36.2, U4.14
- new net: C22.1, R36.2, R50.1, U4.14
Other:
- note added: "C_f = 10nF como filtro pasa bajos profuce una frecuencia de corte de F_c = 482[Hz]"
- note added: "C_f = 1nF para aplanar la respuesta de C_i = 1nF parasito"
- note added: "C_f = 30pF para aplanar la respuesta de C_i = 1nF parasito"
- note added: "C_f=1.5nF para aplanar la respuesta de C_i=1nF parasito"
- note added: "C_f=10nF como filtro pasa bajos profuce una frecuencia de corte de F_c=15.9[kHz]"
- note added: "C_f=200pF Como cota inferior del filtro pasa bajos F_c=23.6[kHz] --> Media geometrica entre 1600Hz y 350kHz"
- note added: "C_f=674pF Como cota inferior del filtro pasa bajos F_c=23.6[kHz] --> Media geometrica entre 1600Hz y 350kHz"
- note added: "Calculado"
- note removed: "NUEVO"
- moved on the sheet: C24, C30, R12, R25, R49, U5D

Commit message: Falta por aprobar errores en la etapa de amplificación
Parts:
- R12: value 100K -> 1K
- R25: value 330k -> 24k
Other:
- note added: "C_f = 303pF para aplanar la respuesta de C_i = 1nF parasito"
- note added: "C_f = 42pF para aplanar la respuesta de C_i = 1nF parasito"
- note added: "C_f=10nF como filtro pasa bajos profuce una frecuencia de corte de F_c=48[Hz] !!!!!!!!!"
- note added: "C_f=10nF como filtro pasa bajos profuce una frecuencia de corte de F_c=663[Hz] !?!?!?"
- note added: "C_f=20pF Como cota inferior del filtro pasa bajos F_c=23.6[kHz] --> Media geometrica entre 1600Hz y 350kHz"
- note added: "C_f=281pF Como cota inferior del filtro pasa bajos F_c=23.6[kHz] --> Media geometrica entre 1600Hz y 350kHz"
- note added: "La etapa de realimentación negativa tiene el mismo criterio que el LPF"
- note added: "Los diodos tienen capacitancia en su polarización inversa, la resistencia de 120[Ohm] anterior evita este problema."
- note added: "Pasa de tener A_v = 3.3 = 330k/100k a tener A_v = 24 = 24k/1k Esto hay que revisarlo y buscar alternativa"
- note added: "R=100[k] C=10[nF] F_c=159[Hz] Cambia a R=10[k] C=10[nF] F_c=1591[Hz]"
- note added: "R_f = 24k R_i = 1k"
- note added: "R_f = 330k R_i = 100k"
- note removed: "Calculado"
- note removed: "R=100[k] C=10[nF] F_c=159[Hz] R=10[k] C=10[nF] F_c=1591[Hz]"
- note removed: "Resistencias (120 Ohm) entre etapas que contengan capacitor INA --> HPF HPF --> BSF AMP_inv --> Nivelador"
- note removed: "Se agregaron capacitores de 10nF a cada filtro El valor real del capacitor hay que calcularlo y aprobarlo en simulación"
- moved on the sheet: C1, C14, C15, C16, C17, C18, C19, C2, C22, C25, C26, C31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

Commit message: termino de esqurmatico
Parts:
- R25: value 24k -> 1k
Other:
- note added: "CORREGIDO"
- note added: "C_f = 6.4[nF] Como cota inferior del filtro pasa bajos F_c = 23.6[kHz] --> Media geometrica entre 1600Hz y 350kHz"
- note added: "C_f=10nF como filtro pasa bajos profuce una frecuencia de corte de F_c=16[kHz]"
- note added: "R_f = 1k R_i = 1k"
- note added: "Se deja en una amplificación de A_v = 1 = 1k/1k"
- note removed: "C_f = 303pF para aplanar la respuesta de C_i = 1nF parasito"
- note removed: "C_f = 42pF para aplanar la respuesta de C_i = 1nF parasito"
- note removed: "C_f=10nF como filtro pasa bajos profuce una frecuencia de corte de F_c=48[Hz] !!!!!!!!!"
- note removed: "C_f=10nF como filtro pasa bajos profuce una frecuencia de corte de F_c=663[Hz] !?!?!?"
- note removed: "C_f=20pF Como cota inferior del filtro pasa bajos F_c=23.6[kHz] --> Media geometrica entre 1600Hz y 350kHz"
- note removed: "C_f=281pF Como cota inferior del filtro pasa bajos F_c=23.6[kHz] --> Media geometrica entre 1600Hz y 350kHz"
- note removed: "R_f = 24k R_i = 1k"
- note removed: "R_f = 330k R_i = 100k"
Changed lines of the file:
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@@
 		)
 	)
-	(text "R_f = 24k\nR_i = 1k"
+	(text "Pasa de tener A_v = 3.3 = 330k/100k\na tener A_v = 24 = 24k/1k\nEsto hay que revisarlo y buscar alternativa\n"
 		(exclude_from_sim no)
-		(at 328.93 332.486 0)
+		(at 208.28 376.428 0)
 		(effects
 			(font
 				(size 1.27 1.27)
-				(thickness 0.254)
-				(bold yes)
-			)
-		)
-	)
-	(text "R_f = 330k\nR_i = 100k"
-		(exclude_from_sim no)
-		(at 285.242 339.09 0)
-		(effects
-			(font
-				(size 1.27 1.27)
-				(thickness 0.254)
-				(bold yes)
-			)
-		)
-	)
-	(text "Pasa de tener A_v = 3.3 = 330k/100k\na tener A_v = 24 = 24k/1k\nEsto hay que revisarlo y buscar alternativa"
-		(exclude_from_sim no)
-		(at 210.312 370.586 0)
-		(effects
-			(font
-				(size 2.032 2.032)
-				(thickness 0.254)
-				(bold yes)
-				(color 193 15 15 1)
+				(thickness 0.1588)
 			)
 		)
@@
 		)
 	)
-	(text "C_f = 303pF para aplanar la \nrespuesta de C_i = 1nF parasito "
-		(exclude_from_sim no)
-		(at 285.75 354.584 0)
-		(effects
-			(font
-				(size 0.889 0.889)
-			)
-		)
-	)
 	(text "La etapa de realimentación negativa\ntiene el mismo criterio que el LPF"
 		(exclude_from_sim no)
@@
 		)
 	)
-	(text "C_f=10nF como filtro pasa bajos\nprofuce una frecuencia de corte de\nF_c=5.9[kHz]"
+	(text "SobreFiltrado"
 		(exclude_from_sim no)
-		(at 145.288 270.002 0)
+		(at 286.512 334.264 0)
+		(effects
+			(font
+				(size 1.778 1.778)
+				(thickness 0.3556)
+				(bold yes)
+			)
+		)
+	)
+	(text "C_f=10nF como filtro pasa bajos\nprofuce una frecuencia de corte de\nF_c=16[kHz]"
+		(exclude_from_sim no)
+		(at 286.258 339.852 0)
 		(effects
 			(font
@@
 		)
 	)
-	(text "SobreFiltrado"
+	(text "C_f=10nF como filtro pasa bajos\nprofuce una frecuencia de corte de\nF_c=5.9[kHz]"
 		(exclude_from_sim no)
-		(at 329.692 336.55 0)
+		(at 145.288 270.002 0)
 		(effects
 			(font
-				(size 1.778 1.778)
-				(thickness 0.3556)
-				(bold yes)
+				(size 1.27 1.27)
 			)
 		)
@@
 		)
 	)
+	(text "SubFiltrado"
+		(exclude_from_sim no)
+		(at 285.496 356.616 0)
+		(effects
+			(font
+				(size 1.778 1.778)
+				(thickness 0.3556)
+				(bold yes)
+			)
+		)
+	)
 	(text "SobreFiltrado"
 		(exclude_from_sim no)
@@
 		)
 	)
-	(text "C_f = 42pF para aplanar la \nrespuesta de C_i = 1nF parasito "
-		(exclude_from_sim no)
-		(at 329.692 352.298 0)
-		(effects
-			(font
-				(size 1.27 1.27)
-			)
-		)
-	)
 	(text "C_f=2.5nF Como cota inferior\ndel filtro pasa bajos\nF_c=23.6[kHz] --> Media geometrica entre \n				  1600Hz y 350kHz "
 		(exclude_from_sim no)
@@
 		)
 	)
-	(text "C_f=674pF Como cota inferior\ndel filtro pasa bajos\nF_c=23.6[kHz] --> Media geometrica entre \n				  1600Hz y 350kHz "
+	(text "C_f = 1nF para aplanar la \nrespuesta de C_i = 1nF parasito "
 		(exclude_from_sim no)
-		(at 306.07 245.872 0)
+		(at 286.512 350.012 0)
 		(effects
 			(font
@@
 		)
 	)
-	(text "C_f=281pF Como cota inferior\ndel filtro pasa bajos\nF_c=23.6[kHz] --> Media geometrica entre \n				  1600Hz y 350kHz "
+	(text "C_f=674pF Como cota inferior\ndel filtro pasa bajos\nF_c=23.6[kHz] --> Media geometrica entre \n				  1600Hz y 350kHz "
 		(exclude_from_sim no)
-		(at 329.692 364.49 0)
+		(at 306.07 245.872 0)
 		(effects
 			(font
@@
 		)
 	)
+	(text "CriticamenteFiltrado"
+		(exclude_from_sim no)
+		(at 286.258 345.948 0)
+		(effects
+			(font
+				(size 1.778 1.778)
+				(thickness 0.3556)
+				(bold yes)
+			)
+		)
+	)
 	(text "C_f=1.5nF para aplanar la \nrespuesta de C_i=1nF parasito "
 		(exclude_from_sim no)
@@
 		)
 	)
-	(text "CriticamenteFiltrado"
+	(text "CORREGIDO"
 		(exclude_from_sim no)
-		(at 329.438 348.234 0)
+		(at 208.534 371.094 0)
 		(effects
 			(font
-				(size 1.778 1.778)
-				(thickness 0.3556)
+				(size 1.905 1.905)
+				(thickness 0.381)
 				(bold yes)
 			)
@@
 		)
 	)
-	(text "C_f=20pF Como cota inferior\ndel filtro pasa bajos\nF_c=23.6[kHz] --> Media geometrica entre \n				  1600Hz y 350kHz "
+	(text "Se deja en una amplificación de A_v = 1 = 1k/1k"
 		(exclude_from_sim no)
-		(at 285.75 363.22 0)
+		(at 211.074 382.524 0)
 		(effects
 			(font
-				(size 0.889 0.889)
+				(size 1.905 1.905)
+				(thickness 0.254)
+				(bold yes)
+				(color 10 65 6 1)
 			)
 		)
@@
 		)
 	)
-	(text "C_f=10nF como filtro pasa bajos\nprofuce una frecuencia de corte de\nF_c=663[Hz] !?!?!?"
+	(text "C_f = 6.4[nF] Como cota inferior\ndel filtro pasa bajos\nF_c = 23.6[kHz] --> Media geometrica entre \n				  1600Hz y 350kHz "
 		(exclude_from_sim no)
-		(at 329.438 342.138 0)
+		(at 286.512 362.204 0)
 		(effects
 			(font
 				(size 1.27 1.27)
-				(color 255 8 8 1)
-			)
-		)
-	)
-	(text "C_f=10nF como filtro pasa bajos\nprofuce una frecuencia de corte de\nF_c=48[Hz] !!!!!!!!!"
-		(exclude_from_sim no)
-		(at 285.242 347.218 0)
-		(effects
-			(font
-				(size 0.889 0.889)
-				(color 230 0 0 1)
 			)
 		)
@@
 	(text "SubFiltrado"
 		(exclude_from_sim no)
-		(at 328.676 358.902 0)
+		(at 305.054 240.284 0)
 		(effects
 			(font
@@
 	(text "CriticamenteFiltrado"
 		(exclude_from_sim no)
-		(at 285.496 351.536 0)
-		(effects
-			(font
-				(size 0.889 0.889)
-				(thickness 0.3556)
-				(bold yes)
-			)
-		)
-	)
-	(text "SubFiltrado"
-		(exclude_from_sim no)
-		(at 305.054 240.284 0)
+		(at 305.816 229.616 0)
 		(effects
 			(font
@@
 		)
 	)
-	(text "SubFiltrado"
-		(exclude_from_sim no)
-		(at 284.734 358.648 0)
-		(effects
-			(font
-				(size 0.889 0.889)
-				(thickness 0.3556)
-				(bold yes)
-			)
-		)
-	)
-	(text "SobreFiltrado"
-		(exclude_from_sim no)
-		(at 285.242 343.662 0)
-		(effects
-			(font
-				(size 0.889 0.889)
-				(thickness 0.3556)
-				(bold yes)
-			)
-		)
-	)
-	(text "CriticamenteFiltrado"
+	(text "C_f=3.7nF para aplanar la \nrespuesta de C_i=1nF parasito "
 		(exclude_from_sim no)
-		(at 305.816 229.616 0)
+		(at 147.066 346.202 0)
 		(effects
 			(font
-				(size 1.778 1.778)
-				(thickness 0.3556)
-				(bold yes)
+				(size 1.27 1.27)
 			)
 		)
 	)
-	(text "C_f=3.7nF para aplanar la \nrespuesta de C_i=1nF parasito "
+	(text "R_f = 1k\nR_i = 1k"
 		(exclude_from_sim no)
-		(at 147.066 346.202 0)
+		(at 285.75 330.2 0)
 		(effects
 			(font
 				(size 1.27 1.27)
+				(thickness 0.254)
+				(bold yes)
 			)
 		)
@@
 			)
 		)
-		(property "Value" "24k"
+		(property "Value" "1k"
 			(at 226.314 346.71 90)
 			(show_name no)

Commit message: m
Parts:
- R11: footprint Resistor_SMD:R_0805_2012Metric_Pad1.20x1.40mm_HandSolder -> Resistor_SMD:R_0603_1608Metric_Pad0.98x0.95mm_HandSolder
Changed lines of the file:
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@@
 			)
 		)
-		(property "Footprint" "Resistor_SMD:R_0805_2012Metric_Pad1.20x1.40mm_HandSolder"
+		(property "Footprint" "Resistor_SMD:R_0603_1608Metric_Pad0.98x0.95mm_HandSolder"
 			(at 78.232 293.37 90)
 			(hide yes)
