File: KiCAD/Electrocardiograma.kicad_pcb (KiCad board)
At the start: 2 copper layers, 56.5 x 48.1 mm, 84 parts, among them J1 54-00174, J2 Conn_01x02_Pin, J3 USB_C_Receptacle_PowerOnly_6P, J4 Conn_01x02_Pin, J5 Conn_01x02_Pin, J6 Conn_01x04_Pin, U1 INA823DT, U2 ESP32-C3-WROOM-02, U3 TLV1117-33, U4 TLV4888, U5 TLV4888, U6 TLV1117-ADJ, U7 SC6038, U8 CH224K

Commit message: Schematic Adjustments
Parts:
- added C26: 10nF, Capacitor_SMD:C_0805_2012Metric_Pad1.18x1.45mm_HandSolder, F.Cu at (196.9, 87.0)
- added R45: 120, Resistor_SMD:R_0805_2012Metric_Pad1.20x1.40mm_HandSolder, F.Cu at (197.9, 110.0)
- added R47: 120, Resistor_SMD:R_0805_2012Metric_Pad1.20x1.40mm_HandSolder, F.Cu at (197.9, 112.9)
- added R48: 120, Resistor_SMD:R_0805_2012Metric_Pad1.20x1.40mm_HandSolder, F.Cu at (197.9, 115.9)
- added R49: 120, Resistor_SMD:R_0805_2012Metric_Pad1.20x1.40mm_HandSolder, F.Cu at (197.9, 118.8)
- moved R42 3.35 mm to (188.0, 86.5)
- moved R40 1.73 mm to (153.5, 88.6), turned to 0 degrees
- moved D6 1.50 mm to (188.0, 82.5)
Connections:
- C11 pad 2: /LPF_out -> Net-(C11-Pad2)
- C20 pad 2: /HPF_out -> Net-(C20-Pad2)
- C21 pad 2: /N50Hz_out -> Net-(C21-Pad2)
- C23 pad 2: /LPF_out -> Net-(C11-Pad2)
- C24 pad 2: /Sensing_Out -> Net-(C24-Pad2)
- C5 pad 1: /N50Hz_out -> Net-(C21-Pad2)
- C8 pad 1: /N50Hz_out -> Net-(C21-Pad2)
- R10 pad 2: /N50Hz_out -> Net-(C21-Pad2)
- R14 pad 2: /HPF_out -> Net-(C20-Pad2)
- R17 pad 2: /HPF_out -> Net-(C20-Pad2)
- R21 pad 2: /LPF_out -> Net-(C11-Pad2)
- R25 pad 2: /Sensing_Out -> Net-(C24-Pad2)
- U5 pad 1: /HPF_out -> Net-(C20-Pad2)
- U5 pad 14: /Sensing_Out -> Net-(C24-Pad2)
- U5 pad 7: /N50Hz_out -> Net-(C21-Pad2)
- U5 pad 8: /LPF_out -> Net-(C11-Pad2)
Routing:
- net +3.3V: track 135.6 -> 134.3 mm
- net -BATT_REG: vias 32 -> 33
